File: 8x8_controller/8x8_controller.kicad_pcb (KiCad board)
At the start: 2 copper layers, 71.1 x 71.1 mm, 15 parts, among them J1 PJ-037A, J2 Conn_01x03_Socket, J3 Conn_01x03_Socket

Commit message: Updated library organization
Parts:
- A1: footprint 8x8_controller:Arduino_Nano_Socket -> 8x8_controller_library:Arduino_Nano_Socket
- J1: footprint 8x8_controller:CUI_PJ-037A -> 8x8_controller_library:CUI_PJ-037A
Changed lines of the file:
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@@
 		)
 	)
-	(footprint "8x8_controller:CUI_PJ-037A"
+	(footprint "8x8_controller_library:CUI_PJ-037A"
 		(layer "F.Cu")
 		(at 170.18 113.08 -90)
 		(property "Reference" "J1"
-			(at 2.485784 -6.76712 90)
+			(at 2.485784 -6.76712 -90)
 			(layer "F.SilkS")
 			(effects
@@
 		)
 		(property "Value" "PJ-037A"
-			(at 6.296338 5.776235 90)
+			(at 6.296338 5.776235 -90)
 			(layer "F.Fab")
 			(effects
@@
 			)
 		)
-		(property "Footprint" "8x8_controller:CUI_PJ-037A"
-			(at 0 0 90)
+		(property "Footprint" "8x8_controller_library:CUI_PJ-037A"
+			(at 0 0 -90)
 			(layer "F.Fab")
 			(hide yes)
@@
 		)
 		(property "Datasheet" ""
-			(at 0 0 90)
+			(at 0 0 -90)
 			(layer "F.Fab")
 			(hide yes)
@@
 		)
 		(property "Description" ""
-			(at 0 0 90)
+			(at 0 0 -90)
 			(layer "F.Fab")
 			(hide yes)
@@
 		)
 		(fp_text user "${REFERENCE}"
-			(at 0 2.54 360)
+			(at 0 2.54 0)
 			(layer "F.Fab")
 			(effects
@@
 		)
 	)
-	(footprint "8x8_controller:Arduino_Nano_Socket"
+	(footprint "8x8_controller_library:Arduino_Nano_Socket"
 		(layer "F.Cu")
 		(at 147.32 125.73)
@@
 			)
 		)
-		(property "Footprint" "8x8_controller:Arduino_Nano_Socket"
+		(property "Footprint" "8x8_controller_library:Arduino_Nano_Socket"
 			(at 0 0 0)
 			(layer "F.Fab")
@@
 		)
 		(fp_text user "${REFERENCE}"
-			(at 0 2.54 360)
-			(layer "F.Fab")
-			(effects
+			(at 0 2.54 0)
+			(layer "F.Fab")
+			(effects

Commit message: 1v0 Complete for proto
Parts:
- removed @HOLE0, @HOLE2, @HOLE3, @HOLE5: , 
- added ?: , , F.Cu at (129.3, 72.4)
- added ?: , , F.Cu at (182.5, 108.2)
- added ?: , , F.Cu at (182.5, 72.4)
- added ?: , , F.Cu at (129.3, 107.9)
- added G***: LOGO, 8x8_controller_library:HAZE_8mm_silkscreen, F.Cu at (177.3, 59.9)
- CSMD_1: renamed from C1; footprint Capacitor_SMD:CP_Elec_8x6.7 -> 8x8_controller_library:CAP_EDT476-9H_KEM-L
- CSMD_2: renamed from C3; footprint Capacitor_SMD:CP_Elec_8x6.7 -> 8x8_controller_library:CAP_EDT476-9H_KEM-L
- moved FID3 66.0 mm to (121.8, 58.3)
- moved CSMD_2 46.6 mm to (174.0, 106.0), turned to 0 degrees
- moved CTHT_2 22.9 mm to (172.3, 93.9), turned to 0 degrees
- moved CSMD_1 5.06 mm to (136.3, 64.6)
- moved CTHT_1 2.10 mm to (139.3, 72.2)
- renumbered C2 to CTHT_1, C4 to CTHT_2
Connections:
- CSMD_1 pad 1: unconnected-(C1-Pad1) -> +VDC
- CSMD_1 pad 2: unconnected-(C1-Pad2) -> GND
- CSMD_2 pad 1: unconnected-(C3-Pad1) -> +VDC
- CSMD_2 pad 2: unconnected-(C3-Pad2) -> GND
- CTHT_1 pad 1: unconnected-(C2-Pad1) -> +VDC
- CTHT_1 pad 2: unconnected-(C2-Pad2) -> GND
- CTHT_2 pad 1: unconnected-(C4-Pad1) -> +VDC
- CTHT_2 pad 2: unconnected-(C4-Pad2) -> GND
Routing:
- net unconnected-(A1-RESET-PadRST2): track 0.00 -> 2.28 mm
- net unconnected-(A1-RESET-PadRST1): track 0.00 -> 2.28 mm
- net unconnected-(A1-PadD9): track 0.00 -> 2.28 mm
- net unconnected-(A1-PadD8): track 0.00 -> 2.28 mm
- net unconnected-(A1-PadD7): track 0.00 -> 2.28 mm
- net unconnected-(A1-PadD5): track 0.00 -> 2.28 mm
- net unconnected-(A1-PadD4): track 0.00 -> 2.28 mm
- net unconnected-(A1-PadD10): track 0.00 -> 2.28 mm
- net unconnected-(A1-PadAREF): track 0.00 -> 2.28 mm
- net unconnected-(A1-PadA7): track 0.00 -> 2.28 mm
- net unconnected-(A1-PadA6): track 0.00 -> 2.28 mm
- net unconnected-(A1-PadA3): track 0.00 -> 2.28 mm
- net unconnected-(A1-PadA2): track 0.00 -> 2.28 mm
- net unconnected-(A1-PadA1): track 0.00 -> 2.28 mm
- net unconnected-(A1-PadA0): track 0.00 -> 2.28 mm
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- added copper zone on B.Cu, net GND
- added copper zone on F.Cu, net GND
- removed copper zone on B.Cu, net (none)
- removed copper zone on F.Cu, net (none)
Other:
- board text added: "8x8 Matrix Controller 1v0"
- board text added: "Haze Engineering, LLC"
